File: board/THVD1400D.kicad_sch (KiCad schematic)
At the start: 6 parts, among them U2 THVD1400D

Commit message: Final update
Other:
- moved on the sheet: C6, JP1
Changed lines of the file:
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@@
 (kicad_sch (version 20230121) (generator eeschema)
   (paper "A4")
-  (junction (at 160.655 74.295) (diameter 0) (color 0 0 0 0)
+  (junction (at 161.29 74.93) (diameter 0) (color 0 0 0 0)
   )
   (junction (at 162.56 104.14) (diameter 0) (color 0 0 0 0)
@@
     (stroke (width 0) (type default))
   )
-  (wire (pts (xy 119.38 97.155) (xy 119.38 105.41))
-    (stroke (width 0) (type default))
-  )
-  (wire (pts (xy 111.125 100.33) (xy 132.08 100.33))
-    (stroke (width 0) (type default))
-  )
-  (wire (pts (xy 130.81 97.155) (xy 130.81 102.87))
+  (wire (pts (xy 119.38 97.79) (xy 119.38 105.41))
+    (stroke (width 0) (type default))
+  )
+  (wire (pts (xy 111.76 100.33) (xy 132.08 100.33))
+    (stroke (width 0) (type default))
+  )
+  (wire (pts (xy 130.81 97.79) (xy 130.81 102.87))
     (stroke (width 0) (type default))
   )
@@
     (stroke (width 0) (type default))
   )
-  (wire (pts (xy 111.125 107.95) (xy 132.08 107.95))
-    (stroke (width 0) (type default))
-  )
-  (wire (pts (xy 160.655 73.025) (xy 160.655 74.295))
+  (wire (pts (xy 111.76 107.95) (xy 132.08 107.95))
+    (stroke (width 0) (type default))
+  )
+  (wire (pts (xy 161.29 73.66) (xy 161.29 74.93))
     (stroke (width 0) (type default))
   )
@@
     (stroke (width 0) (type default))
   )
-  (wire (pts (xy 111.125 105.41) (xy 119.38 105.41))
+  (wire (pts (xy 111.76 105.41) (xy 119.38 105.41))
     (stroke (width 0) (type default))
   )
@@
     (stroke (width 0) (type default))
   )
-  (wire (pts (xy 142.24 74.295) (xy 142.24 90.17))
-    (stroke (width 0) (type default))
-  )
-  (wire (pts (xy 160.655 74.295) (xy 160.655 75.565))
+  (wire (pts (xy 142.24 74.93) (xy 142.24 90.17))
+    (stroke (width 0) (type default))
+  )
+  (wire (pts (xy 161.29 74.93) (xy 161.29 76.2))
     (stroke (width 0) (type default))
   )
@@
     (stroke (width 0) (type default))
   )
-  (wire (pts (xy 121.285 97.155) (xy 119.38 97.155))
-    (stroke (width 0) (type default))
-  )
-  (wire (pts (xy 128.905 97.155) (xy 130.81 97.155))
+  (wire (pts (xy 121.92 97.79) (xy 119.38 97.79))
+    (stroke (width 0) (type default))
+  )
+  (wire (pts (xy 129.54 97.79) (xy 130.81 97.79))
     (stroke (width 0) (type default))
   )
@@
     (stroke (width 0) (type default))
   )
-  (wire (pts (xy 160.655 80.645) (xy 160.655 83.185))
+  (wire (pts (xy 161.29 81.28) (xy 161.29 83.82))
     (stroke (width 0) (type default))
   )
@@
     (stroke (width 0) (type default))
   )
-  (wire (pts (xy 142.24 74.295) (xy 160.655 74.295))
+  (wire (pts (xy 142.24 74.93) (xy 161.29 74.93))
     (stroke (width 0) (type default))
   )
@@
     (effects (font (size 1.27 1.27)) (justify left))
   )
-  (hierarchical_label "DE" (shape input) (at 111.125 105.41 180) (fields_autoplaced)
+  (hierarchical_label "DE" (shape input) (at 111.76 105.41 180) (fields_autoplaced)
     (effects (font (size 1.27 1.27)) (justify right))
   )
-  (hierarchical_label "DI" (shape input) (at 111.125 107.95 180) (fields_autoplaced)
+  (hierarchical_label "DI" (shape input) (at 111.76 107.95 180) (fields_autoplaced)
     (effects (font (size 1.27 1.27)) (justify right))
   )
@@
     (effects (font (size 1.27 1.27)) (justify left))
   )
-  (hierarchical_label "RO" (shape output) (at 111.125 100.33 180) (fields_autoplaced)
+  (hierarchical_label "RO" (shape output) (at 111.76 100.33 180) (fields_autoplaced)
     (effects (font (size 1.27 1.27)) (justify right))
   )
-  (symbol (lib_id "power:GND") (at 160.655 83.185 0) (unit 1)
-    (in_bom yes) (on_board yes) (dnp no) (fields_autoplaced)
-    (property "Reference" "#PWR014" (at 160.655 89.535 0)
-      (effects (font (size 1.27 1.27)) hide)
-    )
-    (property "Value" "GND" (at 160.655 88.265 0)
-      (effects (font (size 1.27 1.27)))
-    )
-    (property "Footprint" "" (at 160.655 83.185 0)
-      (effects (font (size 1.27 1.27)) hide)
-    )
-    (property "Datasheet" "" (at 160.655 83.185 0)
+  (symbol (lib_id "power:GND") (at 161.29 83.82 0) (unit 1)
+    (in_bom yes) (on_board yes) (dnp no) (fields_autoplaced)
+    (property "Reference" "#PWR014" (at 161.29 90.17 0)
+      (effects (font (size 1.27 1.27)) hide)
+    )
+    (property "Value" "GND" (at 161.29 88.9 0)
+      (effects (font (size 1.27 1.27)))
+    )
+    (property "Footprint" "" (at 161.29 83.82 0)
+      (effects (font (size 1.27 1.27)) hide)
+    )
+    (property "Datasheet" "" (at 161.29 83.82 0)
       (effects (font (size 1.27 1.27)) hide)
     )
@@
     )
   )
-  (symbol (lib_id "power:+3V3") (at 160.655 73.025 0) (unit 1)
-    (in_bom yes) (on_board yes) (dnp no) (fields_autoplaced)
-    (property "Reference" "#PWR013" (at 160.655 76.835 0)
-      (effects (font (size 1.27 1.27)) hide)
-    )
-    (property "Value" "+3V3" (at 160.655 67.945 0)
-      (effects (font (size 1.27 1.27)))
-    )
-    (property "Footprint" "" (at 160.655 73.025 0)
-      (effects (font (size 1.27 1.27)) hide)
-    )
-    (property "Datasheet" "" (at 160.655 73.025 0)
+  (symbol (lib_id "power:+3V3") (at 161.29 73.66 0) (unit 1)
+    (in_bom yes) (on_board yes) (dnp no) (fields_autoplaced)
+    (property "Reference" "#PWR013" (at 161.29 77.47 0)
+      (effects (font (size 1.27 1.27)) hide)
+    )
+    (property "Value" "+3V3" (at 161.29 68.58 0)
+      (effects (font (size 1.27 1.27)))
+    )
+    (property "Footprint" "" (at 161.29 73.66 0)
+      (effects (font (size 1.27 1.27)) hide)
+    )
+    (property "Datasheet" "" (at 161.29 73.66 0)
       (effects (font (size 1.27 1.27)) hide)
     )
@@
     )
   )
-  (symbol (lib_id "Jumper:SolderJumper_2_Open") (at 125.095 97.155 0) (unit 1)
-    (in_bom yes) (on_board yes) (dnp no) (fields_autoplaced)
-    (property "Reference" "JP1" (at 125.095 91.44 0)
-      (effects (font (size 1.27 1.27)))
-    )
-    (property "Value" "DE/~{RE}" (at 125.095 93.98 0)
-      (effects (font (size 1.27 1.27)))
-    )
-    (property "Footprint" "Jumper:SolderJumper-2_P1.3mm_Open_RoundedPad1.0x1.5mm" (at 125.095 97.155 0)
-      (effects (font (size 1.27 1.27)) hide)
-    )
-    (property "Datasheet" "~" (at 125.095 97.155 0)
+  (symbol (lib_id "Jumper:SolderJumper_2_Open") (at 125.73 97.79 0) (unit 1)
+    (in_bom yes) (on_board yes) (dnp no) (fields_autoplaced)
+    (property "Reference" "JP1" (at 125.73 92.075 0)
+      (effects (font (size 1.27 1.27)))
+    )
+    (property "Value" "DE/~{RE}" (at 125.73 94.615 0)
+      (effects (font (size 1.27 1.27)))
+    )
+    (property "Footprint" "Jumper:SolderJumper-2_P1.3mm_Open_RoundedPad1.0x1.5mm" (at 125.73 97.79 0)
+      (effects (font (size 1.27 1.27)) hide)
+    )
+    (property "Datasheet" "~" (at 125.73 97.79 0)
       (effects (font (size 1.27 1.27)) hide)
     )
@@
     )
   )
-  (symbol (lib_id "Device:C_Small") (at 160.655 78.105 0) (unit 1)
-    (in_bom yes) (on_board yes) (dnp no) (fields_autoplaced)
-    (property "Reference" "C6" (at 163.195 76.8413 0)
-      (effects (font (size 1.27 1.27)) (justify left))
-    )
-    (property "Value" "4.7uF" (at 163.195 79.3813 0)
-      (effects (font (size 1.27 1.27)) (justify left))
-    )
-    (property "Footprint" "Capacitor_SMD:C_0603_1608Metric" (at 160.655 78.105 0)
-      (effects (font (size 1.27 1.27)) hide)
-    )
-    (property "Datasheet" "~" (at 160.655 78.105 0)
-      (effects (font (size 1.27 1.27)) hide)
-    )
+  (symbol (lib_id "Device:C_Small") (at 161.29 78.74 0) (unit 1)
+    (in_bom yes) (on_board yes) (dnp no) (fields_autoplaced)
+    (property "Reference" "C6" (at 163.83 77.4763 0)
+      (effects (font (size 1.27 1.27)) (justify left))
+    )
+    (property "Value" "4.7uF" (at 163.83 80.0163 0)
+      (effects (font (size 1.27 1.27)) (justify left))
+    )
+    (property "Footprint" "Capacitor_SMD:C_0603_1608Metric" (at 161.29 78.74 0)
+      (effects (font (size 1.27 1.27)) hide)
+    )
+    (property "Datasheet" "~" (at 161.29 78.74 0)
+      (effects (font (size 1.27 1.27)) hide)
+    )

Commit message: Update board
Parts:
- removed C8: 4.7uF, Capacitor_SMD:C_0603_1608Metric, symbol Device:C_Small
- removed JP1: DE/~{RE}, Jumper:SolderJumper-2_P1.3mm_Open_RoundedPad1.0x1.5mm, symbol Jumper:SolderJumper_2_Open
- added D5: SM712, Package_TO_SOT_SMD:SOT-23, symbol Diode:SM712_SOT23
- added R3: 4k7, Resistor_SMD:R_0603_1608Metric, symbol Device:R_Small
- R5, R6: footprint Resistor_SMD:R_0603_1608Metric -> Resistor_SMD:R_0805_2012Metric
Connections:
- net DE: now also U2.2 (~{RE}), R3.1
- net GND: now also D5.3 (common), R3.2
- net RS485_A: now also R5.2, D5.2 (A2); no longer R5.1, U2.7 (B)
- net RS485_B: now also D5.1 (A1); no longer U2.6 (A)
- net at R6.1: now also U2.6 (A); no longer R5.2
- new net: R5.1, U2.7 (B)
Other:
- moved on the sheet: C6, R5, R6
