File: board/rs485_temperature.kicad_pcb (KiCad board)
At the start: 4 copper layers, 50 x 28 mm, 43 parts, among them J1 RS485_IN, J3 DS182, J5 STDC14, J6 RS485_OUT, J7 RS485 TERM, J8 I2C, SW1 SW_Push, U1 STM32C011F6Ux, U2 THVD1400D, U3 L6981N33DR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

Commit message: Final update
Parts:
- J1, J6: footprint Connector_PinSocket_2.00mm:PinSocket_1x04_P2.00mm_Vertical -> Connector_PinHeader_2.00mm:PinHeader_1x04_P2.00mm_Vertical
- SW1: footprint Connector_PinHeader_2.54mm:PinHeader_1x02_P2.54mm_Vertical -> Aliexpress:Push_Button_G71Y_3X6X3.5MM
- moved J8 4.64 mm to (154.0, 87.0), turned to 90 degrees
- moved C5 3.50 mm to (161.5, 84.0), turned to 180 degrees
- moved SW1 2.35 mm to (168.0, 84.1), turned to 0 degrees
- moved R2 2.27 mm to (161.5, 85.5), turned to 0 degrees
Routing:
- net /MCU (STMC011F6Ux)/~{RST}: track 23.9 -> 40.9 mm, vias 1 -> 2
- net /MCU (STMC011F6Ux)/I2C_SDA: track 15.3 -> 20.5 mm
- net +3V3: track 114.6 -> 118.8 mm
- net /MCU (STMC011F6Ux)/I2C_SCL: track 22.8 -> 19.4 mm
- net /MCU (STMC011F6Ux)/RCC_OSCX_OUT: track 3.86 -> 5.92 mm
- net GND: track 33.1 -> 34.3 mm, vias 18 -> 20
Other:
- outline, holes or cut-outs redrawn

Commit message: Update board
Parts:
- removed C8: 4.7uF, Capacitor_SMD:C_0603_1608Metric
- removed J8: I2C, Connector_PinHeader_2.54mm:PinHeader_2x02_P2.54mm_Vertical
- removed JP1: DE/~{RE}, Jumper:SolderJumper-2_P1.3mm_Open_RoundedPad1.0x1.5mm
- added D5: SM712, Package_TO_SOT_SMD:SOT-23, F.Cu at (151.0, 102.4)
- added F1: 100mA, Fuse:Fuse_0805_2012Metric, F.Cu at (142.4, 106.0)
- added G1: LiborW_neg_10x10, LiborW:LiborW_neg_5x5, F.Cu at (158.5, 93.4)
- added R3: 4k7, Resistor_SMD:R_0603_1608Metric, F.Cu at (154.7, 90.1)
- J3: value DS182 -> DS18S20; footprint Connector_PinSocket_2.00mm:PinSocket_1x03_P2.00mm_Vertical -> Connector_PinHeader_2.00mm:PinHeader_1x03_P2.00mm_Vertical
- R1, R5: footprint Resistor_SMD:R_0603_1608Metric -> Resistor_SMD:R_0805_2012Metric
- moved J1 6.00 mm to (146.0, 106.0)
- moved U2 4.83 mm to (151.0, 92.3)
- moved R5 4.61 mm to (149.8, 98.3), turned to -90 degrees
- moved R1 4.37 mm to (152.2, 98.3)
- moved C6 4.32 mm to (154.7, 95.6), turned to -90 degrees
- moved J6 3.00 mm to (155.0, 106.0)
- moved R6 2.48 mm to (161.1, 102.0)
- moved J7 2.46 mm to (158.0, 100.0), turned to 0 degrees
Connections:
- J1 pad 1: +24V -> /PWR
- J6 pad 1: +24V -> /PWR
- R1 pad 1: /RS485 (THVD1400D)/RS485_A -> Net-(U2-B)
- R1 pad 2: Net-(C8-Pad1) -> /RS485 (THVD1400D)/RS485_A
- R5 pad 1: Net-(C8-Pad1) -> Net-(U2-A)
- U2 pad 2: Net-(JP1-B) -> /MCU (STMC011F6Ux)/USART1_DE
- U2 pad 6: /RS485 (THVD1400D)/RS485_B -> Net-(U2-A)
- U2 pad 7: /RS485 (THVD1400D)/RS485_A -> Net-(U2-B)
Routing:
- net /MCU (STMC011F6Ux)/I2C_SDA: track 20.5 -> 0.00 mm, vias 1 -> 0
- net /MCU (STMC011F6Ux)/I2C_SCL: track 19.4 -> 0.00 mm, vias 1 -> 0
- net /PWR: track 0.00 -> 14.3 mm
- net +24V: track 13.4 -> 0.00 mm
- net /RS485 (THVD1400D)/RS485_A: track 33.3 -> 20.7 mm
- net /RS485 (THVD1400D)/RS485_B: track 33.3 -> 22.9 mm
- net Net-(JP1-B): track 6.50 -> 0.00 mm
- net /MCU (STMC011F6Ux)/USART1_DE: track 32.0 -> 26.0 mm
- net /MCU (STMC011F6Ux)/USART1_RX: track 25.9 -> 30.9 mm
- net /MCU (STMC011F6Ux)/USART1_TX: track 38.7 -> 42.4 mm
- net Net-(C8-Pad1): track 3.04 -> 0.00 mm
- net Net-(U2-B): track 0.00 -> 2.85 mm
- net Net-(U2-A): track 0.00 -> 2.85 mm
- net GND: track 34.3 -> 33.1 mm, vias 20 -> 33
- net +3V3: track 118.8 -> 119.6 mm
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Other:
- board text added: "+"
- board text added: "-"
- board text added: "A"
- board text added: "B"
- board text added: "D"
- board text added: "RS485 Temperature Sensor v2023/07, r0 serial:"
