File: board/rs485_temperature.kicad_sch (KiCad schematic)
At the start: 16 parts, among them J1 I2C, J1 RS485_IN, J1 RS485_OUT, J3 DS182, J7 RS485 TERM

Commit message: Final update
Parts:
- H1, H2, H3, H4, J3: now left out of the parts list
- J1: footprint Connector_PinSocket_2.00mm:PinSocket_1x04_P2.00mm_Vertical -> Connector_PinHeader_2.00mm:PinHeader_1x04_P2.00mm_Vertical; now left out of the parts list
- J6: renamed from J1; footprint Connector_PinSocket_2.00mm:PinSocket_1x04_P2.00mm_Vertical -> Connector_PinHeader_2.00mm:PinHeader_1x04_P2.00mm_Vertical; now left out of the parts list
- J8: renamed from J1; now left out of the parts list
Changed lines of the file:
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@@
   )
   (symbol (lib_id "Mechanical:MountingHole") (at 21.59 190.5 0) (unit 1)
-    (in_bom yes) (on_board yes) (dnp no) (fields_autoplaced)
+    (in_bom no) (on_board yes) (dnp no) (fields_autoplaced)
     (property "Reference" "H2" (at 24.13 189.23 0)
       (effects (font (size 1.27 1.27)) (justify left))
@@
   )
   (symbol (lib_id "Connector_Generic:Conn_01x04") (at 45.72 104.14 0) (mirror y) (unit 1)
-    (in_bom yes) (on_board yes) (dnp no)
-    (property "Reference" "J1" (at 45.72 115.57 0)
+    (in_bom no) (on_board yes) (dnp no)
+    (property "Reference" "J8" (at 45.72 115.57 0)
       (effects (font (size 1.27 1.27)))
     )
@@
   )
   (symbol (lib_id "Mechanical:MountingHole") (at 29.21 190.5 0) (unit 1)
-    (in_bom yes) (on_board yes) (dnp no) (fields_autoplaced)
+    (in_bom no) (on_board yes) (dnp no) (fields_autoplaced)
     (property "Reference" "H3" (at 31.75 189.23 0)
       (effects (font (size 1.27 1.27)) (justify left))
@@
   )
   (symbol (lib_id "Connector_Generic:Conn_01x04") (at 45.72 48.26 0) (mirror y) (unit 1)
-    (in_bom yes) (on_board yes) (dnp no)
+    (in_bom no) (on_board yes) (dnp no)
     (property "Reference" "J1" (at 45.72 59.69 0)
       (effects (font (size 1.27 1.27)))
@@
       (effects (font (size 1.27 1.27)))
     )
-    (property "Footprint" "Connector_PinSocket_2.00mm:PinSocket_1x04_P2.00mm_Vertical" (at 45.72 48.26 0)
+    (property "Footprint" "Connector_PinHeader_2.00mm:PinHeader_1x04_P2.00mm_Vertical" (at 45.72 48.26 0)
       (effects (font (size 1.27 1.27)) hide)
     )
@@
   )
   (symbol (lib_id "Connector_Generic:Conn_01x04") (at 45.72 72.39 0) (mirror y) (unit 1)
-    (in_bom yes) (on_board yes) (dnp no)
-    (property "Reference" "J1" (at 45.72 83.82 0)
+    (in_bom no) (on_board yes) (dnp no)
+    (property "Reference" "J6" (at 45.72 83.82 0)
       (effects (font (size 1.27 1.27)))
     )
@@
       (effects (font (size 1.27 1.27)))
     )
-    (property "Footprint" "Connector_PinSocket_2.00mm:PinSocket_1x04_P2.00mm_Vertical" (at 45.72 72.39 0)
+    (property "Footprint" "Connector_PinHeader_2.00mm:PinHeader_1x04_P2.00mm_Vertical" (at 45.72 72.39 0)
       (effects (font (size 1.27 1.27)) hide)
     )
@@
   (symbol (lib_id "power:GND") (at 201.93 62.23 0) (unit 1)
     (in_bom yes) (on_board yes) (dnp no) (fields_autoplaced)
-    (property "Reference" "#PWR038" (at 201.93 68.58 0)
+    (property "Reference" "#PWR017" (at 201.93 68.58 0)
       (effects (font (size 1.27 1.27)) hide)
     )
@@
   (symbol (lib_id "power:GND") (at 53.34 124.46 0) (unit 1)
     (in_bom yes) (on_board yes) (dnp no) (fields_autoplaced)
-    (property "Reference" "#PWR034" (at 53.34 130.81 0)
+    (property "Reference" "#PWR022" (at 53.34 130.81 0)
       (effects (font (size 1.27 1.27)) hide)
     )
@@
   )
   (symbol (lib_id "Mechanical:MountingHole") (at 29.21 185.42 0) (unit 1)
-    (in_bom yes) (on_board yes) (dnp no) (fields_autoplaced)
+    (in_bom no) (on_board yes) (dnp no) (fields_autoplaced)
     (property "Reference" "H4" (at 31.75 184.15 0)
       (effects (font (size 1.27 1.27)) (justify left))
@@
   (symbol (lib_id "power:+3V3") (at 57.15 96.52 0) (unit 1)
     (in_bom yes) (on_board yes) (dnp no) (fields_autoplaced)
-    (property "Reference" "#PWR037" (at 57.15 100.33 0)
+    (property "Reference" "#PWR021" (at 57.15 100.33 0)
       (effects (font (size 1.27 1.27)) hide)
     )
@@
   (symbol (lib_id "power:GND") (at 219.71 43.18 0) (unit 1)
     (in_bom yes) (on_board yes) (dnp no) (fields_autoplaced)
-    (property "Reference" "#PWR038" (at 219.71 49.53 0)
+    (property "Reference" "#PWR019" (at 219.71 49.53 0)
       (effects (font (size 1.27 1.27)) hide)
     )
@@
   (symbol (lib_id "power:+3V3") (at 219.71 31.75 0) (unit 1)
     (in_bom yes) (on_board yes) (dnp no) (fields_autoplaced)
-    (property "Reference" "#PWR037" (at 219.71 35.56 0)
+    (property "Reference" "#PWR016" (at 219.71 35.56 0)
       (effects (font (size 1.27 1.27)) hide)
     )
@@
   )
   (symbol (lib_id "Connector_Generic:Conn_01x03") (at 209.55 52.07 0) (unit 1)
-    (in_bom yes) (on_board yes) (dnp no) (fields_autoplaced)
+    (in_bom no) (on_board yes) (dnp no) (fields_autoplaced)
     (property "Reference" "J3" (at 212.09 50.8 0)
       (effects (font (size 1.27 1.27)) (justify left))
@@
   )
   (symbol (lib_id "Mechanical:MountingHole") (at 21.59 185.42 0) (unit 1)
-    (in_bom yes) (on_board yes) (dnp no) (fields_autoplaced)
+    (in_bom no) (on_board yes) (dnp no) (fields_autoplaced)
     (property "Reference" "H1" (at 24.13 184.15 0)
       (effects (font (size 1.27 1.27)) (justify left))

Commit message: Update board
Parts:
- removed J8: I2C, Connector_PinHeader_2.54mm:PinHeader_2x02_P2.54mm_Vertical, symbol Connector_Generic:Conn_01x04
- added F1: 100mA, Fuse:Fuse_0805_2012Metric, symbol Device:Polyfuse_Small
- added G1: LiborW_neg_10x10, LiborW:LiborW_neg_5x5, symbol LiborW:LiborW_neg_10x10
- J3: value DS182 -> DS18S20; footprint Connector_PinSocket_2.00mm:PinSocket_1x03_P2.00mm_Vertical -> Connector_PinHeader_2.00mm:PinHeader_1x03_P2.00mm_Vertical; Label (none) -> DS18S20
Connections:
- net +24V: now also F1.2; no longer J1.1 (Pin_1), J6.1 (Pin_1)
- new net PWR: F1.1, J1.1 (Pin_1), J6.1 (Pin_1)
- no-connect marks 0 -> 2
Changed lines of the file:
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@@
   (junction (at 190.5 52.07) (diameter 0) (color 0 0 0 0)
   )
-  (junction (at 53.34 109.22) (diameter 0) (color 0 0 0 0)
-  )
   (junction (at 219.71 35.56) (diameter 0) (color 0 0 0 0)
   )
@@
   (junction (at 64.77 50.8) (diameter 0) (color 0 0 0 0)
   )
+  (no_connect (at 134.62 104.14))
+  (no_connect (at 134.62 101.6))
+  (wire (pts (xy 74.93 45.72) (xy 67.31 45.72))
+    (stroke (width 0) (type default))
+  )
   (wire (pts (xy 172.72 93.98) (xy 186.69 93.98))
     (stroke (width 0) (type default))
@@
     (stroke (width 0) (type default))
   )
-  (wire (pts (xy 50.8 109.22) (xy 53.34 109.22))
-    (stroke (width 0) (type default))
-  )
   (wire (pts (xy 50.8 45.72) (xy 57.15 45.72))
     (stroke (width 0) (type default))
@@
     (stroke (width 0) (type default))
   )
-  (wire (pts (xy 53.34 72.39) (xy 53.34 109.22))
-    (stroke (width 0) (type default))
-  )
-  (wire (pts (xy 50.8 101.6) (xy 134.62 101.6))
+  (wire (pts (xy 53.34 72.39) (xy 53.34 124.46))
     (stroke (width 0) (type default))
   )
@@
     (stroke (width 0) (type default))
   )
+  (wire (pts (xy 62.23 45.72) (xy 57.15 45.72))
+    (stroke (width 0) (type default))
+  )
   (wire (pts (xy 57.15 45.72) (xy 57.15 69.85))
     (stroke (width 0) (type default))
@@
     (stroke (width 0) (type default))
   )
-  (wire (pts (xy 53.34 109.22) (xy 53.34 124.46))
-    (stroke (width 0) (type default))
-  )
   (wire (pts (xy 190.5 49.53) (xy 190.5 52.07))
     (stroke (width 0) (type default))
@@
     (stroke (width 0) (type default))
   )
-  (wire (pts (xy 57.15 96.52) (xy 57.15 106.68))
-    (stroke (width 0) (type default))
-  )
-  (wire (pts (xy 50.8 106.68) (xy 57.15 106.68))
-    (stroke (width 0) (type default))
-  )
   (wire (pts (xy 172.72 83.82) (xy 186.69 83.82))
     (stroke (width 0) (type default))
@@
     (stroke (width 0) (type default))
   )
-  (wire (pts (xy 50.8 104.14) (xy 134.62 104.14))
-    (stroke (width 0) (type default))
-  )
   (wire (pts (xy 201.93 93.98) (xy 201.93 100.33))
     (stroke (width 0) (type default))
@@
     (stroke (width 0) (type default))
   )
-  (wire (pts (xy 57.15 39.37) (xy 57.15 45.72))
+  (wire (pts (xy 74.93 39.37) (xy 74.93 45.72))
     (stroke (width 0) (type default))
   )
   (wire (pts (xy 219.71 31.75) (xy 219.71 35.56))
     (stroke (width 0) (type default))
+  )
+  (label "PWR" (at 52.07 45.72 0) (fields_autoplaced)
+    (effects (font (size 1.27 1.27)) (justify left bottom))
+  )
+  (symbol (lib_id "LiborW:LiborW_neg_10x10") (at 184.15 173.99 0) (unit 1)
+    (in_bom no) (on_board yes) (dnp no) (fields_autoplaced)
+    (property "Reference" "G1" (at 184.15 169.6468 0)
+      (effects (font (size 1.27 1.27)) hide)
+    )
+    (property "Value" "LiborW_neg_10x10" (at 184.15 178.3332 0)
+      (effects (font (size 1.27 1.27)) hide)
+    )
+    (property "Footprint" "LiborW:LiborW_neg_5x5" (at 184.15 173.99 0)
+      (effects (font (size 1.27 1.27)) hide)
+    )
+    (property "Datasheet" "" (at 184.15 173.99 0)
+      (effects (font (size 1.27 1.27)) hide)
+    )
+    (instances
+      (project "rs485_temperature"
+        (path "/b2de72b7-bd7d-4616-84ab-7321f2f03a54"
+          (reference "G1") (unit 1)
+        )
+      )
+    )
   )
   (symbol (lib_id "Device:LED_Small") (at 196.85 93.98 180) (unit 1)
@@
     )
   )
-  (symbol (lib_id "Connector_Generic:Conn_01x04") (at 45.72 104.14 0) (mirror y) (unit 1)
-    (in_bom no) (on_board yes) (dnp no)
-    (property "Reference" "J8" (at 45.72 115.57 0)
-      (effects (font (size 1.27 1.27)))
-    )
-    (property "Value" "I2C" (at 45.72 113.03 0)
-      (effects (font (size 1.27 1.27)))
-    )
-    (property "Footprint" "Connector_PinHeader_2.54mm:PinHeader_2x02_P2.54mm_Vertical" (at 45.72 104.14 0)
-      (effects (font (size 1.27 1.27)) hide)
-    )
-    (property "Datasheet" "~" (at 45.72 104.14 0)
-      (effects (font (size 1.27 1.27)) hide)
-    )
-    (pin "1")
-    (pin "2")
-    (pin "3")
-    (pin "4")
-    (instances
-      (project "rs485_temperature"
-        (path "/b2de72b7-bd7d-4616-84ab-7321f2f03a54"
-          (reference "J8") (unit 1)
-        )
-      )
-    )
-  )
   (symbol (lib_id "Connector_Generic:Conn_01x02") (at 67.31 90.17 270) (unit 1)
     (in_bom yes) (on_board yes) (dnp no)
@@
     )
   )
+  (symbol (lib_id "Device:Polyfuse_Small") (at 64.77 45.72 90) (unit 1)
+    (in_bom yes) (on_board yes) (dnp no) (fields_autoplaced)
+    (property "Reference" "F1" (at 64.77 39.37 90)
+      (effects (font (size 1.27 1.27)))
+    )
+    (property "Value" "100mA" (at 64.77 41.91 90)
+      (effects (font (size 1.27 1.27)))
+    )
+    (property "Footprint" "Fuse:Fuse_0805_2012Metric" (at 69.85 44.45 0)
+      (effects (font (size 1.27 1.27)) (justify left) hide)
+    )
+    (property "Datasheet" "~" (at 64.77 45.72 0)
+      (effects (font (size 1.27 1.27)) hide)
+    )
+    (pin "1")
+    (pin "2")
+    (instances
+      (project "rs485_temperature"
+        (path "/b2de72b7-bd7d-4616-84ab-7321f2f03a54"
+          (reference "F1") (unit 1)
+        )
+      )
+    )
+  )
   (symbol (lib_id "Mechanical:MountingHole") (at 29.21 185.42 0) (unit 1)
     (in_bom no) (on_board yes) (dnp no) (fields_autoplaced)
@@
     )
   )
-  (symbol (lib_id "power:+3V3") (at 57.15 96.52 0) (unit 1)
-    (in_bom yes) (on_board yes) (dnp no) (fields_autoplaced)
-    (property "Reference" "#PWR021" (at 57.15 100.33 0)
-      (effects (font (size 1.27 1.27)) hide)
-    )
-    (property "Value" "+3V3" (at 57.15 91.44 0)
-      (effects (font (size 1.27 1.27)))
-    )
-    (property "Footprint" "" (at 57.15 96.52 0)
-      (effects (font (size 1.27 1.27)) hide)
-    )
-    (property "Datasheet" "" (at 57.15 96.52 0)
-      (effects (font (size 1.27 1.27)) hide)
-    )
-    (pin "1")
-    (instances
-      (project "rs485_temperature"
-        (path "/b2de72b7-bd7d-4616-84ab-7321f2f03a54"
-          (reference "#PWR021") (unit 1)
-        )
-      )
-    )
-  )
-  (symbol (lib_id "power:+24V") (at 57.15 39.37 0) (unit 1)
-    (in_bom yes) (on_board yes) (dnp no) (fields_autoplaced)
-    (property "Reference" "#PWR024" (at 57.15 43.18 0)
-      (effects (font (size 1.27 1.27)) hide)
-    )
-    (property "Value" "+24V" (at 57.15 33.655 0)
-      (effects (font (size 1.27 1.27)))
-    )
-    (property "Footprint" "" (at 57.15 39.37 0)
-      (effects (font (size 1.27 1.27)) hide)
-    )
-    (property "Datasheet" "" (at 57.15 39.37 0)
+  (symbol (lib_id "power:+24V") (at 74.93 39.37 0) (unit 1)
+    (in_bom yes) (on_board yes) (dnp no) (fields_autoplaced)
+    (property "Reference" "#PWR024" (at 74.93 43.18 0)
+      (effects (font (size 1.27 1.27)) hide)
+    )
+    (property "Value" "+24V" (at 74.93 33.655 0)
+      (effects (font (size 1.27 1.27)))
+    )
+    (property "Footprint" "" (at 74.93 39.37 0)
+      (effects (font (size 1.27 1.27)) hide)
+    )
+    (property "Datasheet" "" (at 74.93 39.37 0)
       (effects (font (size 1.27 1.27)) hide)
     )
@@
       (effects (font (size 1.27 1.27)) (justify left))
     )
-    (property "Value" "DS182" (at 212.09 53.34 0)
-      (effects (font (size 1.27 1.27)) (justify left))
-    )
-    (property "Footprint" "Connector_PinSocket_2.00mm:PinSocket_1x03_P2.00mm_Vertical" (at 209.55 52.07 0)
+    (property "Value" "DS18S20" (at 212.09 53.34 0)
+      (effects (font (size 1.27 1.27)) (justify left))
+    )
+    (property "Footprint" "Connector_PinHeader_2.00mm:PinHeader_1x03_P2.00mm_Vertical" (at 209.55 52.07 0)
       (effects (font (size 1.27 1.27)) hide)
     )
@@
       (effects (font (size 1.27 1.27)) hide)
     )
+    (property "Label" "DS18S20" (at 209.55 52.07 0)
+      (effects (font (size 1.27 1.27)) hide)
+    )
